File: template_board/can.kicad_sch (KiCad schematic)
At the start: 19 parts, among them IC1 TJA1044GTK_3Z, IC2 TJA1044GTK_3Z, J7 RJ45_LED_Shielded, J8 RJ45_LED_Shielded, SW5 SW_DIP_x02

Commit message: u5 wip
Parts:
- removed C44, C45: 10n, Capacitor_SMD:C_0402_1005Metric, symbol Device:C
- removed J7, J8: RJ45_LED_Shielded, Connector_RJ:RJ45_Amphenol_RJHSE538X, symbol Connector:RJ45_LED_Shielded
- removed R48, R49, R52, R53: 1k, Resistor_SMD:R_0402_1005Metric, symbol Device:R
- removed R50, R51: 33k, Resistor_SMD:R_0402_1005Metric, symbol Device:R
Other:
- note removed: "PASS THROUYH BUS CONENCTOR"
- note removed: "min 200V"
