File: template_board/MCU.kicad_sch (KiCad schematic)
At the start: 31 parts, among them SW1 SW_Push, U5 STM32U575RITx, X3 Q13FC1350000400, X4 X322512MSB4SI

Commit message: [schematics] complete lora board
Connections:
- net LORA.MISO: now reaches U5.10 (PC2)
- net GPIO8: now reaches U5.11 (PC3)
- net GPIO16: now reaches U5.14 (PA0)
- net GPIO24: now reaches U5.15 (PA1)
- net GPIO1: now reaches U5.16 (PA2)
- net GPIO9: now reaches U5.17 (PA3)
- net GPIO0: now reaches U5.2 (PC13)
- net GPIO17: now reaches U5.20 (PA4)
- net LORA_DIO0: now reaches U5.21 (PA5)
- net LORA_DIO1: now reaches U5.22 (PA6)
- net LORA_DIO2: now reaches U5.23 (PA7)
- net LORA_DIO3: now reaches U5.24 (PC4)
- net LORA_DIO4: now reaches U5.25 (PC5)
- net LORA_DIO5: now reaches U5.26 (PB0)
- net LORA.CS: now reaches U5.27 (PB1)
- net ~{LORA_RESET}: now reaches U5.28 (PB2)
- net LORA.CLK: now reaches U5.29 (PB10)
- net GPIO18: now reaches U5.33 (PB12)
- net GPIO26: now reaches U5.34 (PB13)
- net GPIO3: now reaches U5.35 (PB14)
- net GPIO11: now reaches U5.36 (PB15)
- net GPIO19: now reaches U5.37 (PC6)
- net GPIO27: now reaches U5.38 (PC7)
- net GPIO4: now reaches U5.39 (PC8)
- net GPIO12: now reaches U5.40 (PC9)
- net GPIO10: now reaches U5.50 (PA15)
- net GPIO2: now reaches U5.53 (PC12)
- net GPIO25: now reaches U5.54 (PD2)
- net LORA.MOSI: now reaches U5.9 (PC1)
- no-connect marks 29 -> 0
