File: template_board/lora.kicad_sch (KiCad schematic)
At the start: 4 parts, among them J2 Conn_Coaxial, U8 Ai-Thinker-Ra-01

Commit message: fixed USB\Power leyout , added proper RF rules adn paths
Connections:
- net RF: now reaches J2.1 (In), U8.1 (ANT)
Changed lines of the file:
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@@
+		)
+	)
+	(label "RF"
+		(at 132.08 71.12 0)
+		(effects
+			(font
+				(size 1.27 1.27)
+			)
+			(justify left bottom)
 		)
 	)
